File: hardware/flappy6502.kicad_sch (KiCad schematic)
At the start: 34 parts, among them J1 LCD (SmartElex ST7789P3), J2 5V 2A in, SW1 RESET, SW2 FLAP, U1 R6502 (NMOS), U2 AT28C64B-15 ($E000-$FFFF), U3 HY62CT08081E ($0000-$7FFF), U4 74LS00 decoder, U5 74LS161 LCD latch ($8000), U6 74LS161 clock divider, U7 74LS04, Y1 10 MHz

Commit message: Schematic: one A3 sheet with every connection wired (rows + channels, risers, A/D buses), netlist-verified
Parts:
- J1: value LCD (SmartElex ST7789P3) -> LCD ST7789P3
- J2: value 5V 2A in -> 5V in
- U1: value R6502 (NMOS) -> R6502 (NMOS CPU)
- U2: value AT28C64B-15 ($E000-$FFFF) -> AT28C64B ROM $E000
- U3: value HY62CT08081E ($0000-$7FFF) -> HY62C SRAM $0000
- U4: value 74LS00 decoder -> 74LS00
- U5: value 74LS161 LCD latch ($8000) -> 74LS161 LCD latch $8000
- U6: value 74LS161 clock divider -> 74LS161 clock /8
Connections:
- net CLK10M: no longer names the net of U6.2 (CP), U7.12
- net LCD_CS: no longer names the net of J1.4 (Pin_4), U5.11 (Q3)
- net LCD_DC: no longer names the net of J1.6 (Pin_6), U5.12 (Q2)
- net LCD_RST: no longer names the net of J1.2 (Pin_2), J1.7 (Pin_7), U7.4
- net LCD_SCL: no longer names the net of J1.5 (Pin_5), U5.13 (Q1)
- net LCD_SDA: no longer names the net of J1.1 (Pin_1), U5.14 (Q0)
- net RDY: no longer names the net of R3.2, U1.2 (RDY)
- net RSTB: no longer names the net of U7.2, U7.3
- net SO: no longer names the net of R6.2, U1.38 (SO)
- net ~{IOSEL}: no longer names the net of U4.6, U5.9 (~{PE})
- net ~{IRQ}: no longer names the net of R4.2, U1.4 (~{IRQ})
Other:
- note removed: "CPU clock PHI0 = U6 QC (1.25 MHz) or QD pin 11 (625 kHz). C4 sits at U5 pin 2."
- note removed: "Decoupling: C9-C15 100n at each IC (U1-U7); C8 10u at the CPU."
- note removed: "J1 pins: 1 SDA 2 RST 3 TE 4 CS 5 SCL 6 DC 7 EN 8 GND 9 VCC"
- note removed: "LCD rule: never feed the module 5 V; RST and EN come from U7 (low during reset)."
- note removed: "Memory map: RAM $0000-$7FFF, LCD latch $8000 (bit0 SDA, bit1 SCL, bit2 DC, bit3 CS), ROM $E000-$FFFF"
- note removed: "flappy6502 - R6502 + 28C64 + 32K SRAM + 74LS logic -> ST7789 LCD (bit-banged SPI)"
